Commit message: steven WIP IK fixes

File: assets/koch_follower.urdf (robot description, URDF)
Before this commit: robot robot, 7 links, 6 joints
Joints:
- joint joint_1: limit lower=-3.14 upper=3.14 effort=0.5 velocity=100 -> lower=-1.5 upper=1.5 effort=0.5 velocity=100
- joint joint_2: limit lower=-3.14 upper=3.14 effort=0.5 velocity=100 -> lower=-1.5 upper=1.5 effort=0.5 velocity=100
- joint joint_3: limit lower=-3.14 upper=3.14 effort=0.5 velocity=100 -> lower=-1.50 upper=1.50 effort=0.5 velocity=100
- joint joint_4: limit lower=-3.14 upper=3.14 effort=0.5 velocity=100 -> lower=-1.5 upper=1.5 effort=0.5 velocity=100
- joint joint_5: limit lower=-3.14 upper=3.14 effort=0.5 velocity=100 -> lower=-1.5 upper=1.5 effort=0.5 velocity=100

Commit message: MCP support

File: assets/koch_follower.urdf (robot description, URDF)
Before this commit: robot robot, 7 links, 6 joints
Links:
- added link ee_frame
Joints:
- added joint ee_frame_joint: type fixed, parent link_6, child ee_frame, origin xyz=0 0 0 rpy=0.785398163397 0 0
